File: PCB/BMS_SMD_SpiceSim/BMS_SMD_SpiceSim.kicad_sch (KiCad schematic)
At the start: 11 parts, among them U1 INA180A1

Commit message: WIP: recover pre-repair project reorganization
Restores reorganized source, tests, GUI harnesses, and current development files. Eleven unit tests pass; measurement-report and integration tests remain work in progress.
Connections:
- net Load: no longer R2.2, R4.2, V2.1
- new net: R2.2, R4.2, V2.1
Other:
- note added: "ADC Current A2D count = ~32000"
- note removed: "ADC A2D count = ~32000"
- moved on the sheet: R4
Changed lines of the file:
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@@
 		)
 	)
-	(text "ADC A2D count = ~32000"
+	(text "ADC Current A2D count = ~32000"
 		(exclude_from_sim no)
 		(at 163.068 79.502 0)
@@
 	)
 	(junction
+		(at 118.11 92.71)
+		(diameter 0)
+		(color 0 0 0 0)
+	)
+	(junction
+		(at 208.28 52.07)
+		(diameter 0)
+		(color 0 0 0 0)
+	)
+	(junction
+		(at 198.12 91.44)
+		(diameter 0)
+		(color 0 0 0 0)
+	)
+	(junction
+		(at 138.43 85.09)
+		(diameter 0)
+		(color 0 0 0 0)
+	)
+	(junction
+		(at 205.74 86.36)
+		(diameter 0)
+		(color 0 0 0 0)
+	)
+	(junction
+		(at 210.82 91.44)
+		(diameter 0)
+		(color 0 0 0 0)
+	)
+	(junction
+		(at 203.2 86.36)
+		(diameter 0)
+		(color 0 0 0 0)
+	)
+	(junction
+		(at 210.82 93.98)
+		(diameter 0)
+		(color 0 0 0 0)
+	)
+	(junction
+		(at 198.12 106.68)
+		(diameter 0)
+		(color 0 0 0 0)
+	)
+	(junction
 		(at 163.83 88.9)
 		(diameter 0)
@@
 	)
 	(junction
-		(at 118.11 92.71)
-		(diameter 0)
-		(color 0 0 0 0)
-	)
-	(junction
-		(at 208.28 52.07)
-		(diameter 0)
-		(color 0 0 0 0)
-	)
-	(junction
-		(at 198.12 91.44)
-		(diameter 0)
-		(color 0 0 0 0)
-	)
-	(junction
-		(at 200.66 86.36)
-		(diameter 0)
-		(color 0 0 0 0)
-	)
-	(junction
-		(at 138.43 85.09)
-		(diameter 0)
-		(color 0 0 0 0)
-	)
-	(junction
-		(at 205.74 86.36)
-		(diameter 0)
-		(color 0 0 0 0)
-	)
-	(junction
-		(at 210.82 91.44)
-		(diameter 0)
-		(color 0 0 0 0)
-	)
-	(junction
-		(at 210.82 93.98)
-		(diameter 0)
-		(color 0 0 0 0)
-	)
-	(junction
-		(at 198.12 106.68)
-		(diameter 0)
-		(color 0 0 0 0)
-	)
-	(junction
 		(at 210.82 106.68)
 		(diameter 0)
@@
 	(wire
 		(pts
-			(xy 208.28 52.07) (xy 208.28 76.2)
-		)
-		(stroke
-			(width 0.508)
-			(type default)
-		)
-	)
-	(wire
-		(pts
-			(xy 198.12 86.36) (xy 200.66 86.36)
+			(xy 208.28 52.07) (xy 208.28 74.93)
+		)
+		(stroke
+			(width 0.508)
+			(type default)
+		)
+	)
+	(wire
+		(pts
+			(xy 198.12 86.36) (xy 203.2 86.36)
 		)
 		(stroke
@@
 	(wire
 		(pts
-			(xy 200.66 83.82) (xy 200.66 86.36)
+			(xy 203.2 82.55) (xy 203.2 86.36)
 		)
 		(stroke
@@
 	(wire
 		(pts
-			(xy 200.66 76.2) (xy 208.28 76.2)
-		)
-		(stroke
-			(width 0.508)
-			(type default)
-		)
-	)
-	(wire
-		(pts
 			(xy 210.82 91.44) (xy 210.82 92.71)
 		)
@@
 	(wire
 		(pts
-			(xy 200.66 86.36) (xy 205.74 86.36)
-		)
-		(stroke
-			(width 0.508)
-			(type default)
-		)
-	)
-	(wire
-		(pts
 			(xy 171.45 88.9) (xy 182.88 88.9)
 		)
@@
 	(wire
 		(pts
+			(xy 203.2 86.36) (xy 205.74 86.36)
+		)
+		(stroke
+			(width 0.508)
+			(type default)
+		)
+	)
+	(wire
+		(pts
 			(xy 162.56 87.63) (xy 163.83 88.9)
 		)
@@
 		(pts
 			(xy 210.82 93.98) (xy 210.82 106.68)
+		)
+		(stroke
+			(width 0.508)
+			(type default)
+		)
+	)
+	(wire
+		(pts
+			(xy 203.2 74.93) (xy 208.28 74.93)
 		)
 		(stroke
@@
 	)
 	(label "Load"
-		(at 200.66 76.2 0)
+		(at 200.66 74.93 0)
 		(effects
 			(font
@@
 	)
 	(label "Load"
-		(at 200.66 76.2 0)
+		(at 200.66 74.93 0)
 		(effects
 			(font
@@
 	(symbol
 		(lib_id "Device:R")
-		(at 200.66 80.01 180)
+		(at 203.2 78.74 180)
 		(unit 1)
 		(body_style 1)
@@
 		(dnp no)
 		(property "Reference" "R4"
-			(at 203.2 78.7399 0)
+			(at 205.74 77.4699 0)
 			(show_name no)
 			(do_not_autoplace no)
@@
 		)
 		(property "Value" "11.95"
-			(at 200.66 82.804 90)
+			(at 203.2 80.264 90)
 			(show_name no)
 			(do_not_autoplace no)
@@
 		)
 		(property "Footprint" "Resistor_SMD:R_1210_3225Metric_Pad1.30x2.65mm_HandSolder"
-			(at 202.438 80.01 90)
+			(at 204.978 78.74 90)
 			(hide yes)
 			(show_name no)
@@
 		)
 		(property "Datasheet" ""
-			(at 200.66 80.01 0)
+			(at 203.2 78.74 0)
 			(hide yes)
 			(show_name no)
@@
 		)
 		(property "Description" "Resistor"
-			(at 200.66 80.01 0)
+			(at 203.2 78.74 0)
 			(hide yes)
 			(show_name no)
@@
 		)
 		(property "Sim.Params" ""
-			(at 200.66 80.01 0)
-			(hide yes)
-			(show_name no)
+			(at 203.2 78.74 0)
+			(hide yes)
+			(show_name no)
